Commit message: Stop laser_joint yawing the Livox frame 90 degrees
laser_joint carried rpy="0 0 -pi/2", added in perseus-v3's 31015e3 "for
improved alignment", while the comment above it still said the joint
"adds no rotation of its own". The comment described the intent; the yaw
was aligning the mesh.

It is not a cosmetic setting. base_link -> livox_frame resolved to
roll -45, pitch 0, yaw -90 instead of the intended pitch 45, and
fast_lio composes T_map_base = T_map_imu * T_imu_lidar * T_lidar_base
with lid_frame -> base_frame read from TF, so the yaw went straight into
the pose it reports for base_link. On the real robot base_link started 90
degrees off odom the moment localisation came up. Gravity alignment could
not absorb it, since an accelerometer constrains roll and pitch only,
which is why disabling gravity_align_en changed nothing.

In simulation the same joint orients the Gazebo gpu_lidar and IMU, which
attach to livox_frame by reference with no pose of their own, so the
simulated sensor was twisted the same way.

The -pi/2 is folded into the visual and inertial origins instead, so the
mesh renders exactly as it does today, and the comment now says why the
joint must stay unrotated.

Co-Authored-By: Claude Opus 5 (1M context) <noreply@anthropic.com>

File: src/perseus_description/urdf/sensor_mount.urdf.xacro (robot description, xacro)
@@ -57,10 +57,10 @@
     <link name="${prefix}livox_frame">
       <inertial>
-        <origin xyz="0 0.0 0.0" rpy="${pi/2} 0.0 ${pi}"/>
+        <origin xyz="0 0.0 0.0" rpy="${pi/2} 0.0 ${pi/2}"/>
         <mass value="${livox_mass}"/>
         <xacro:box_inertia m="${livox_mass}" x="${livox_length}" y="${livox_radius}" z="${livox_radius}"/>
       </inertial>
       <visual>
-        <origin xyz="0 0.0 -0.02" rpy="${pi/2} 0.0 ${pi}"/>
+        <origin xyz="0 0.0 -0.02" rpy="${pi/2} 0.0 ${pi/2}"/>
         <geometry>
           <mesh scale="1.0 1.0 1.0" filename="file://$(find perseus_description)/meshes/mid-360.dae"/>
@@ -80,9 +80,16 @@
       extrinsic in the fast_lio config is internal to the sensor housing and is unaffected
       by how the housing is mounted.
+      Do not add a rotation here to make the mesh line up. This joint is what says where the
+      sensor points, and fast_lio composes the robot's pose as
+      T_map_base = T_map_imu * T_imu_lidar * T_lidar_base, reading lid_frame -> base_frame
+      straight out of TF, so a yaw added here lands in base_link's reported orientation.
+      A -pi/2 put here for mesh alignment is exactly why base_link once started 90 degrees
+      off odom, and gravity alignment cannot absorb it, because an accelerometer constrains
+      roll and pitch only. Mesh alignment belongs on the <visual> origin above.
     -->
     <joint name="${prefix}laser_joint" type="fixed">
       <parent link="${prefix}livox_base"/>
       <child link="${prefix}livox_frame"/>
-      <origin xyz="${-0.038} 0.0 0.064" rpy="${0.0} 0.0 ${-pi/2}"/>
+      <origin xyz="${-0.038} 0.0 0.064" rpy="0.0 0.0 0.0"/>
     </joint>
     <!-- RealSense D455, on the front face of the mast, looking straight ahead -->
