Commit message: Model the Livox IMU offset instead of putting the IMU on livox_frame
The simulated IMU was attached to livox_frame, so in Gazebo it sat exactly on the
LiDAR origin. The real MID-360 has its IMU 4.4 cm inside the housing, and
perseus-v3's description now states that offset on a livox_imu_joint so the LIO
configs can stop each carrying their own copy of it.

Mirroring the joint here, and moving the imu sensor onto the new frame, closes
two gaps at once. The simulator matches the sensor it is standing in for, and
anything reading the extrinsic out of the robot description gets the same answer
in Gazebo as on the robot -- BIEVR-LIO's calibration.from_tf being the immediate
case, which otherwise had to be given a separate identity extrinsic for
simulation, or would hang waiting for a livox_imu_frame that did not exist.

The link is a pure frame: no visual, no collision, no inertial. sdformat lumps it
into base_link along with every other fixed-joint child, which is what should
happen -- the sensor moves with it and its pose is composed on the way.

Verified by converting the expanded description with `gz sdf -p`: the lidar_imu
sensor comes out at (0.618965, 0.02329, 0.694149) relative to base_link, which is
livox_frame's position plus Ry(45 deg) applied to (0.011, 0.02329, -0.04412), and
reports gz_frame_id livox_imu_frame. Not yet run in Gazebo itself.

File: src/perseus_description/urdf/sensor_mount.urdf.xacro (robot description, xacro)
@@ -93,4 +93,25 @@
       <origin xyz="${-0.038} 0.0 0.064" rpy="0.0 0.0 0.0"/>
     </joint>
+    <!--
+      The IMU inside the Livox housing, and where the Gazebo imu sensor is attached (see
+      sensors.urdf.xacro). A pure frame: no visual, no collision, no inertial, because
+      nothing about the robot's mass or appearance depends on it.
+      The MID-360 datasheet puts the IMU at (11.0, 23.29, -44.12) mm from the LiDAR origin,
+      in LiDAR coordinates, with no rotation between them. Modelling it here rather than
+      leaving the simulated IMU sitting exactly on livox_frame does two things: the
+      simulator matches the real sensor, and BIEVR-LIO can read the extrinsic back out of
+      TF (calibration.from_tf) in simulation exactly as it does on the robot, instead of
+      needing a separate identity extrinsic stated in the sim config.
+      Kept identical to the same joint in perseus-v3's description package, which is the
+      copy the real robot runs.
+      Note the sign. The LIO configs express this extrinsic the other way round, as the
+      LiDAR origin in IMU coordinates, so they carry the negation of these numbers.
+    -->
+    <link name="${prefix}livox_imu_frame"/>
+    <joint name="${prefix}livox_imu_joint" type="fixed">
+      <parent link="${prefix}livox_frame"/>
+      <child link="${prefix}livox_imu_frame"/>
+      <origin xyz="0.011 0.02329 ${-0.04412}" rpy="0.0 0.0 0.0"/>
+    </joint>
     <!-- RealSense D455, on the front face of the mast, looking straight ahead -->
     <xacro:sensor_d455 parent="${prefix}sensor_mount" name="camera" use_nominal_extrinsics="true">

File: src/perseus_description/urdf/sensors.urdf.xacro (robot description, xacro)
@@ -46,5 +46,12 @@
   </sensor>
 </gazebo>
-<gazebo reference="${prefix}livox_frame">
+<!--
+  The IMU is attached to livox_imu_frame, not to livox_frame: it lives 4.4 cm inside the
+  housing from the LiDAR origin, and sensor_mount.urdf.xacro now says so. Attaching it here
+  is what makes that offset real in simulation rather than just present in TF, so anything
+  that reads the LiDAR-IMU extrinsic out of the description gets the same answer in Gazebo
+  as on the robot.
+-->
+<gazebo reference="${prefix}livox_imu_frame">
     <material>Gazebo/Grey</material>
     <sensor name="${prefix}lidar_imu" type="imu">
@@ -56,5 +63,5 @@
         <topic>/scan_3d/imu</topic>
         <!-- Add frame id to imu sensor (achieving correct frame association)-->
-        <gz_frame_id>${prefix}livox_frame</gz_frame_id>
+        <gz_frame_id>${prefix}livox_imu_frame</gz_frame_id>
     </sensor>
 </gazebo>
