Commit message: Mount the bucket frame under the chassis, not on the deck
The frame's rails bolt to the underside of the chassis. The previous value put
them flat on the deck instead, sitting the whole attachment 220 mm too high.

The chassis link origin is the centre of its front face at the bottom, so the
chassis floor is chassis z = 0; putting the rail top face (frame z 0.038) flush
with it gives bucket_mount_z = 0 - (0.038 - 0.213) = 0.175.

Rails now sit at chassis z -0.020..0.000 (base_link 0.330..0.350) and the gantry
at base_link 0.255..0.555 - hanging 95 mm below the chassis floor with 255 mm of
ground clearance against a 150 mm wheel radius.

This also resolves the sensor-mast interference that was logged as a known
issue. The gantry top now clears the Livox at base_link 0.700 by 145 mm.
Measured on the horizontal LiDAR ring:

  no bucket          240 returns,   0 blocked at the 0.1 m minimum
  bucket, deck mount 307 returns,  78 blocked (~40% of the ring lost)
  bucket, under-slung 239 returns,  0 blocked, 45 in 0.15-1 m

The 45 remaining are the arms and bucket genuinely in the forward-down view,
which is true of the real machine; a crop-box self-filter is the fix for that,
not a model change.

Ram loop closure re-verified after the move: still 0.02 mm worst case over the
workspace. Lift, tilt and all six ram joints track; drives without tipping.

Co-Authored-By: Claude Opus 5 (1M context) <noreply@anthropic.com>
Claude-Session: https://claude.ai/code/session_01297Spm5F3sYbgKetBbzuBf

File: src/perseus_description/urdf/bucket.urdf.xacro (robot description, xacro)
@@ -72,17 +72,19 @@
   <xacro:property name="bucket_density" value="2700.0"/>
   <!-- ══ Where the attachment sits on the rover ═══════════════════════════
-       DERIVED, but check it against the real machine.
        The frame's two rearward rails run 243 mm back from the gantry at
-       z = 0.018..0.038 in frame coordinates, 390 mm apart. The rover chassis
-       is 450 mm wide with its deck at chassis z = 0.2, so the rails land on
-       the deck just inside its edges - that is plainly how this bolts on, and
-       it fixes both x and z:
-         z: deck top 0.200 + (arm pivot 0.213 - rail underside 0.018) = 0.395
+       z = 0.018..0.038 in frame coordinates, 390 mm apart. They bolt to the
+       UNDERSIDE of the chassis, so the rail top face sits flush with the
+       chassis floor. The chassis link origin is the centre of its front face
+       at the bottom, so that floor is chassis z = 0:
+         z: 0 - (rail top 0.038 - arm pivot 0.213) = 0.175
          x: gantry front face 17 mm ahead of the chassis front face = 0.0591
-       Note this puts the gantry around the sensor mast - see the warning at
-       the bottom of this file. -->
+       That puts the rails at chassis z -0.020..0.000 (base_link 0.330..0.350)
+       and the gantry at base_link 0.255..0.555 - hanging 95 mm below the
+       chassis floor, with 255 mm of ground clearance against a 150 mm wheel
+       radius. It also drops the gantry top clear of the Livox at base_link
+       0.700 by 145 mm, which an earlier deck-mounted guess did not. -->
   <xacro:property name="bucket_mount_x" value="0.0591"/>
   <xacro:property name="bucket_mount_y" value="0.0"/>
-  <xacro:property name="bucket_mount_z" value="0.395"/>
+  <xacro:property name="bucket_mount_z" value="0.175"/>
   <!-- ══ Linkage geometry ════════════════════════════════════════════════
        All MEASURED, by forward-kinematicking the export's mate transforms
@@ -613,13 +615,9 @@
     </gazebo>
     <!--
-      ⚠ The gantry stands where the sensor mast is.
-      With the mount above, the gantry occupies base_link x 0.600..0.617,
-      z 0.473..0.773. The Livox sits at base_link (0.600, 0, 0.700) and the
-      D455 at (0.600, 0, 0.600) - both inside the gantry's 410 x 300 window
-      rather than inside a beam, so nothing is buried in solid metal, but the
-      LiDAR does look out through the frame and will return hits off its
-      members. That is true of the real rover too, so it is left as it is
-      rather than quietly moved. If you want them separated, change
-      bucket_mount_x/z here - nothing else depends on them.
+      Sensor clearance: the gantry occupies base_link x 0.600..0.617,
+      z 0.255..0.555. The Livox at (0.600, 0, 0.700) and the D455 at
+      (0.600, 0, 0.600) both clear its top. The bucket itself is still in the
+      LiDAR's forward-down view when the arms are raised, which is true of the
+      real machine as well.
     -->
   </xacro:macro>
