Commit message: Sync sensor mount URDF with perseus-v3
Match the finalised mast description from perseus-v3: add the livox_base
plate link with its lidar_base.dae mesh, reparent laser_joint onto it so
the sensor inherits the plate tilt, and apply the tilt once at
livox_base_joint. Rename livox_pitch to lidar_angle to match.

livox_frame moves from sensors.urdf.xacro into sensor_mount.urdf.xacro,
next to the mast it is mounted on. The Gazebo gpu_lidar and IMU sensors
stay in sensors.urdf.xacro and still reference the link by name.

Remove the 2D LIDAR (laser_2d_frame, its joint, properties and Gazebo
block); the hardware is not on the rover and the frame was unused.

Simulation-only divergences are preserved: the perseus_description
package paths, the black material on the Livox visual, and the
deliberately disabled Gazebo D455 cameras.

Meshes are installed per-file by symlink, so lidar_base.dae and
sensor_mount.dae need a rebuild before they resolve.

File: src/perseus_description/urdf/perseus.urdf.xacro (robot description, xacro)
@@ -42,8 +42,5 @@
     <xacro:property name="bar_width" value="0.03"/>
     <xacro:property name="bar_height" value="0.03"/>
-    <!-- 2D and 3D LIDAR Properties -->
-    <xacro:property name="laser_2d_mass" value="0.1"/>
-    <xacro:property name="laser_2d_radius" value="0.04"/>
-    <xacro:property name="laser_2d_length" value="0.04"/>
+    <!-- 3D LIDAR Properties -->
     <xacro:property name="livox_mass" value="0.2"/>
     <xacro:property name="livox_radius" value="0.04"/>
@@ -59,6 +56,8 @@
     <xacro:property name="sensor_mount_y_offset" value="0.0"/>
     <xacro:property name="sensor_mount_z_offset" value="${chassis_height + 0.05}"/>
-    <!-- nose-down tilt of the Livox: positive pitch swings its +x axis towards -z -->
-    <xacro:property name="livox_pitch" value="${pi/4}"/>
+    <!-- nose-down tilt of the Livox base plate, applied at livox_base_joint in
+         sensor_mount.urdf.xacro: positive pitch swings its +x axis towards -z. The
+         sensor is fixed to the plate, so this aims the LiDAR. Zero leaves it level. -->
+    <xacro:property name="lidar_angle" value="${pi/4}"/>
     <!-- ADD COMPONENTS -->
     <xacro:include filename="$(find perseus_description)/urdf/inertia_macros.xacro"/>
@@ -95,9 +94,4 @@
     <!-- Livox and RealSense both hang off the mast: see sensor_mount.urdf.xacro -->
     <xacro:sensor_mount prefix="${prefix}"/>
-    <joint name="${prefix}laser_2d_joint" type="fixed">
-      <parent link="${prefix}chassis"/>
-      <child link="${prefix}laser_2d_frame"/>
-      <origin xyz="-0.15 0 0.25" rpy="0 0 0"/>
-    </joint>
   </xacro:macro>
 </robot>

File: src/perseus_description/urdf/sensor_mount.urdf.xacro (robot description, xacro)
@@ -7,6 +7,6 @@
     extends backwards in -x and upwards in +z from that origin. "Front of the chassis,
     a bit above" is therefore x near 0 and z a little over chassis_height.
-    Both sensors hang off sensor_mount rather than off chassis, so re-siting the mast
-    only means changing sensor_mount_*_offset.
+    Both sensors hang off sensor_mount rather than off chassis (the Livox through
+    livox_base), so re-siting the mast only means changing sensor_mount_*_offset.
   -->
   <xacro:macro name="sensor_mount" params="prefix:=^">
@@ -17,4 +17,10 @@
         <xacro:box_inertia m="${sensor_mount_mass}" x="${sensor_mount_length}" y="${sensor_mount_width}" z="${sensor_mount_height}"/>
       </inertial>
+      <visual>
+        <origin xyz="${-0.023} ${0.005} ${-0.035}" rpy="0.0 0.0 ${pi/2}"/>
+        <geometry>
+          <mesh scale="1.0 1.0 1.0" filename="file://$(find perseus_description)/meshes/sensor_mount.dae"/>
+        </geometry>
+      </visual>
     </link>
     <joint name="${prefix}sensor_mount_joint" type="fixed">
@@ -24,17 +30,63 @@
     </joint>
     <!--
-      Livox MID-360, on top of the mast and pitched nose-down by livox_pitch.
-      A positive pitch about +y takes the sensor +x axis towards -z, so this points the
-      LiDAR forwards and down. The IMU-LiDAR extrinsic in the fast_lio config is internal
-      to the sensor housing and is unaffected by how the housing is mounted.
+      Plate on top of the mast that the Livox bolts onto. lidar_angle is applied here, and
+      the sensor is fixed to the plate, so the two tilt together: a positive pitch about +y
+      takes the plate, and with it the sensor +x axis, towards -z, pointing the LiDAR
+      forwards and down. Re-aiming the LiDAR means changing lidar_angle and nothing else.
+    -->
+    <link name="${prefix}livox_base">
+      <visual>
+        <origin xyz="${-0.082} 0.0 ${0.002}" rpy="${pi/2} 0.0 ${pi}"/>
+        <geometry>
+          <mesh scale="1.0 1.0 1.0" filename="file://$(find perseus_description)/meshes/lidar_base.dae"/>
+        </geometry>
+      </visual>
+    </link>
+    <joint name="${prefix}livox_base_joint" type="fixed">
+      <parent link="${prefix}sensor_mount"/>
+      <child link="${prefix}livox_base"/>
+      <origin xyz="0.024 0.0 0.061" rpy="0.0 ${lidar_angle} 0.0"/>
+    </joint>
+    <!--
+      Livox MID-360 itself. The mesh and the collision cylinder are offset down by 20 mm
+      because the sensor frame sits above the housing floor; the rpy on the visual only
+      aligns the exported mesh with that frame.
+      The Gazebo gpu_lidar and IMU sensors that drive this link live in
+      sensors.urdf.xacro, which references it by name.
+    -->
+    <link name="${prefix}livox_frame">
+      <inertial>
+        <origin xyz="0 0.0 0.0" rpy="${pi/2} 0.0 ${pi}"/>
+        <mass value="${livox_mass}"/>
+        <xacro:box_inertia m="${livox_mass}" x="${livox_length}" y="${livox_radius}" z="${livox_radius}"/>
+      </inertial>
+      <visual>
+        <origin xyz="0 0.0 -0.02" rpy="${pi/2} 0.0 ${pi}"/>
+        <geometry>
+          <mesh scale="1.0 1.0 1.0" filename="file://$(find perseus_description)/meshes/mid-360.dae"/>
+        </geometry>
+        <material name="black"/>
+      </visual>
+      <collision>
+        <origin xyz="0 0.0 -0.02" rpy="0.0 0.0 0.0"/>
+        <geometry>
+          <cylinder radius="${livox_radius}" length="${livox_length}"/>
+        </geometry>
+      </collision>
+    </link>
+    <!--
+      Livox MID-360, seated on livox_base. The joint only offsets it across the plate and
+      adds no rotation of its own, so the sensor inherits the plate's tilt. The IMU-LiDAR
+      extrinsic in the fast_lio config is internal to the sensor housing and is unaffected
+      by how the housing is mounted.
     -->
     <joint name="${prefix}laser_joint" type="fixed">
-      <parent link="${prefix}sensor_mount"/>
+      <parent link="${prefix}livox_base"/>
       <child link="${prefix}livox_frame"/>
-      <origin xyz="0.0 0.0 0.1" rpy="0.0 ${livox_pitch} 0.0"/>
+      <origin xyz="${-0.038} 0.0 0.064" rpy="${0.0} 0.0 ${-pi/2}"/>
     </joint>
     <!-- RealSense D455, on the front face of the mast, looking straight ahead -->
     <xacro:sensor_d455 parent="${prefix}sensor_mount" name="camera" use_nominal_extrinsics="true">
-      <origin xyz="0.0 0.0 0.0" rpy="0.0 0.0 0.0"/>
+      <origin xyz="0.035 0.0 0.006" rpy="0.0 0.0 0.0"/>
     </xacro:sensor_d455>
     <!--

File: src/perseus_description/urdf/sensors.urdf.xacro (robot description, xacro)
@@ -1,47 +1,9 @@
 <?xml version="1.0"?>
 <robot name="lidar" xmlns:xacro="http://ros.org/wiki/xacro">
-<!-- 3D LIDAR (Existing - Livox MID-360) -->
-<link name="${prefix}livox_frame">
-    <inertial>
-        <origin xyz="0 0.0 0.0" rpy="${pi/2} 0.0 ${pi}"/>
-        <mass value="${livox_mass}"/>
-        <xacro:box_inertia m="${livox_mass}" x="${livox_length}" y="${livox_radius}" z="${livox_radius}"/>
-    </inertial>
-    <visual>
-        <origin xyz="0 0.0 -0.02" rpy="${pi/2} 0.0 ${pi}"/>
-        <geometry>
-            <mesh scale="1.0 1.0  1.0" filename="file://$(find perseus_description)/meshes/mid-360.dae"/>
-        </geometry>
-        <material name="black"/>
-    </visual>
-    <collision>
-        <origin xyz="0 0.0 -0.02" rpy="0.0 0.0 0.0"/>
-        <geometry>
-            <cylinder radius="${livox_radius}" length="${livox_length}"/>
-        </geometry>
-    </collision>
-</link>
-<!-- 2D LIDAR -->
-<link name="${prefix}laser_2d_frame">
-    <inertial>
-        <origin xyz="0 0 0"/>
-        <mass value="${laser_2d_mass}"/>
-        <xacro:box_inertia m="${laser_2d_mass}" x="${laser_2d_length}" y="${laser_2d_radius}" z="${laser_2d_radius}"/>
-    </inertial>
-    <visual>
-        <origin xyz="0 0 0"/>
-        <geometry>
-            <cylinder radius="${laser_2d_radius}" length="${laser_2d_length}"/>
-        </geometry>
-        <material name="blue">
-            <color rgba="0.0 0.0 1.0 1.0"/>
-        </material>
-    </visual>
-    <collision>
-        <geometry>
-            <cylinder radius="0.04" length="0.04"/>
-        </geometry>
-    </collision>
-</link>
+<!--
+  Gazebo sensors for the Livox MID-360. The livox_frame link itself is declared in
+  sensor_mount.urdf.xacro, next to the mast it is mounted on; these blocks only attach
+  simulated hardware to it by name.
+-->
 <!-- Simulating the Livox MID-360 -->
 <gazebo reference="${prefix}livox_frame">
@@ -84,19 +46,4 @@
   </sensor>
 </gazebo>
-<!-- 2D LIDAR SENSOR (Traditional 2D Laser Scanner) -->
-<gazebo reference="${prefix}laser_2d_frame">
-  <material>
-    <ambient>0.0 0.0 1.0 1</ambient>
-    <diffuse>0.0 0.0 1.0 1</diffuse>
-    <specular>0.0 0.0 1.0 1</specular>
-  </material>
-  <!--
-    No gpu_lidar sensor here on purpose. A 360 deg gpu_lidar costs roughly 400 ms
-    per frame on this machine regardless of ray count, and a second one drops the
-    real-time factor to ~0.2 without adding anything SLAM needs. The link is kept
-    so the TF tree and rviz configs are unchanged; re-add a <sensor> block here if
-    a 2D scan is ever actually required.
-  -->
-</gazebo>
 <gazebo reference="${prefix}livox_frame">
     <material>Gazebo/Grey</material>

Commit message: Move base_link 0.2 m back from the chassis front face
chassis_joint placed base_link a full chassis_length (0.6 m) ahead of the
chassis origin. perseus-v3 uses a fixed 0.2 m instead, which is what the
bucket mount offsets in bucket.urdf.xacro are measured against.

Taken from perseus-v3 252429c, where this line changed as part of adding the
bucket mount; split out here so the geometry change is visible on its own.

File: src/perseus_description/urdf/perseus.urdf.xacro (robot description, xacro)
@@ -75,5 +75,5 @@
     <link name="${prefix}base_link"/>
     <joint name="${prefix}chassis_joint" type="fixed"> <!-- Joint Connect base_link and chassis -->
-      <origin xyz="${chassis_length} 0.0 ${chassis_z_offset}" rpy="0.0 0.0 0.0"/>
+      <origin xyz="${0.2} 0.0 ${chassis_z_offset}" rpy="0.0 0.0 0.0"/>
       <parent link="${prefix}base_link"/>
       <child link="${prefix}chassis"/>
