Commit message: fix(urdf): sync perseus-v3 sensor mount and footprint changes
- sensor_mount_y_offset 0.0 -> 0.015 and lidar_angle pi/4 -> 7pi/36.
- laser_joint yaw -pi/2 (the real Livox mounting), with the mesh yaw pi/2 -> pi
  on the visual and inertial origins so the drawn model is unchanged.
- Drop the static base_footprint link: flat_footprint_broadcaster publishes
  odom -> base_footprint, and a second parent makes TF reject the frame.

Sim-only parts (file:// mesh paths, bucket.gazebo.xacro, Gazebo sensors) are kept.

Co-Authored-By: Claude Opus 5.5 <noreply@anthropic.com>

File: src/perseus_description/urdf/perseus.urdf.xacro (robot description, xacro)
@@ -54,10 +54,10 @@
          front and z above chassis_height clears the deck -->
     <xacro:property name="sensor_mount_x_offset" value="0.0"/>
-    <xacro:property name="sensor_mount_y_offset" value="0.0"/>
+    <xacro:property name="sensor_mount_y_offset" value="0.015"/>
     <xacro:property name="sensor_mount_z_offset" value="${chassis_height + 0.05}"/>
     <!-- nose-down tilt of the Livox base plate, applied at livox_base_joint in
          sensor_mount.urdf.xacro: positive pitch swings its +x axis towards -z. The
          sensor is fixed to the plate, so this aims the LiDAR. Zero leaves it level. -->
-    <xacro:property name="lidar_angle" value="${pi/4}"/>
+    <xacro:property name="lidar_angle" value="${7*pi/36}"/>
     <!-- ADD COMPONENTS -->
     <xacro:include filename="$(find perseus_description)/urdf/inertia_macros.xacro"/>
@@ -80,10 +80,11 @@
       <child link="${prefix}chassis"/>
     </joint>
-    <link name="${prefix}base_footprint"/>
-    <joint name="base_footprint_joint" type="fixed">
-        <parent link="${prefix}base_link"/>
-        <child link="${prefix}base_footprint"/>
-        <origin xyz="0 0 0" rpy="0 0 0"/>
-    </joint>
+    <!--
+      No base_footprint link here on purpose. footprint_broadcaster's
+      flat_footprint_broadcaster publishes odom -> base_footprint at runtime, and a
+      static base_link -> base_footprint from robot_state_publisher would give the frame
+      a second parent, which TF rejects. The frame is produced by that node, not by the
+      model.
+    -->
     <!-- ADD 2 ROCKERS (INCLUDING 4 MOTORS + 4 WHEELS) -->
     <xacro:rocker prefix="" side="left"/>

File: src/perseus_description/urdf/sensor_mount.urdf.xacro (robot description, xacro)
@@ -57,10 +57,10 @@
     <link name="${prefix}livox_frame">
       <inertial>
-        <origin xyz="0 0.0 0.0" rpy="${pi/2} 0.0 ${pi/2}"/>
+        <origin xyz="0 0.0 0.0" rpy="${pi/2} 0.0 ${pi}"/>
         <mass value="${livox_mass}"/>
         <xacro:box_inertia m="${livox_mass}" x="${livox_length}" y="${livox_radius}" z="${livox_radius}"/>
       </inertial>
       <visual>
-        <origin xyz="0 0.0 -0.02" rpy="${pi/2} 0.0 ${pi/2}"/>
+        <origin xyz="0 0.0 -0.02" rpy="${pi/2} 0.0 ${pi}"/>
         <geometry>
           <mesh scale="1.0 1.0 1.0" filename="file://$(find perseus_description)/meshes/mid-360.dae"/>
@@ -78,18 +78,26 @@
       Livox MID-360, seated on livox_base. The joint only offsets it across the plate and
       adds no rotation of its own, so the sensor inherits the plate's tilt. The IMU-LiDAR
-      extrinsic in the fast_lio config is internal to the sensor housing and is unaffected
+      extrinsic (livox_imu_joint below) is internal to the sensor housing and is unaffected
       by how the housing is mounted.
-      Do not add a rotation here to make the mesh line up. This joint is what says where the
-      sensor points, and fast_lio composes the robot's pose as
-      T_map_base = T_map_imu * T_imu_lidar * T_lidar_base, reading lid_frame -> base_frame
-      straight out of TF, so a yaw added here lands in base_link's reported orientation.
-      A -pi/2 put here for mesh alignment is exactly why base_link once started 90 degrees
-      off odom, and gravity alignment cannot absorb it, because an accelerometer constrains
-      roll and pitch only. Mesh alignment belongs on the <visual> origin above.
+      The -pi/2 yaw is not mesh alignment: the sensor is physically seated on the plate
+      rotated a quarter turn, so TF has to say so. livox_ros_driver2 stamps every cloud
+      frame_id: livox_frame, which means this joint's orientation is what orients every
+      point downstream; get it wrong and the whole point cloud is rotated.
+      96a84d2 removed this yaw (PR #17, fix/livox-frame-yaw) to stop base_link starting
+      90 degrees off odom, and that reversed the trade. The LIO does compose
+      T_map_base = T_map_imu * T_imu_lidar * T_lidar_base with livox_frame -> base_link read
+      from TF (BIEVR-LIO's base.odom_in_base), so the yaw does land in base_link's reported
+      orientation (which base.heading_at_base now corrects for), but odom has no
+      absolute yaw reference (see the imu0 notes in autonomy_bringup/config/ekf_config.yaml),
+      so the odom frame is defined by wherever the robot started and a 90 degree offset in it
+      is cosmetic. A rotated point cloud is not. What has to agree is the cloud and the pose,
+      and only keeping the real mounting rotation here achieves that.
+      Mesh alignment is the pi on the <visual> and <inertial> origins above; the two move
+      together, so changing one without the other makes the model lie about the frame.
     -->
     <joint name="${prefix}laser_joint" type="fixed">
       <parent link="${prefix}livox_base"/>
       <child link="${prefix}livox_frame"/>
-      <origin xyz="${-0.038} 0.0 0.064" rpy="0.0 0.0 0.0"/>
+      <origin xyz="${-0.038} 0.0 0.064" rpy="${0.0} 0.0 ${-pi/2}"/>
     </joint>
     <!--
