Commit message: Add regolith digging plugin and boulder obstacles to the Perseus Arc world
- Integrated the RegolithDig plugin for simulating diggable regolith.
- Added multiple boulder models with specific poses and scales to enhance obstacle variability in the simulation.
- Updated the model references to ensure proper loading of boulder assets.

File: src/perseus_description/urdf/bucket.gazebo.xacro (robot description, xacro)
@@ -81,12 +81,24 @@
       <xacro:bucket_ram_follower joint="bucket_ram_jaw_left_extend_joint"   topic="/bucket/ram_jaw/cmd_extend"  kind="extend"/>
     </gazebo>
-    <!-- The cutting edge needs grip to bite rather than skate. -->
+    <!-- The cutting edge needs grip to bite rather than skate.
+         Every bucket collision is on bit 1 only and the regolith bed on bit 0
+         only (Moon_DEM), so the bucket goes INTO the bed instead of resting on
+         it: the RegolithDig world system (perseus_simulation/src/regolith_dig.cpp)
+         carves the bed where the bucket passes and applies the load and cutting
+         drag as forces. Berms are part of the bed, so the bucket passes through
+         those too. Walls and boulders keep the default all-ones mask, so the
+         bucket still hits them. -->
     <gazebo reference="${prefix}bucket_body">
       <mu1>1.0</mu1>
       <mu2>1.0</mu2>
+      <collision><surface><contact><collide_bitmask>0x02</collide_bitmask></contact></surface></collision>
     </gazebo>
     <gazebo reference="${prefix}bucket_lift_arm">
       <mu1>0.6</mu1>
       <mu2>0.6</mu2>
+      <collision><surface><contact><collide_bitmask>0x02</collide_bitmask></contact></surface></collision>
+    </gazebo>
+    <gazebo reference="${prefix}bucket_jaw">
+      <collision><surface><contact><collide_bitmask>0x02</collide_bitmask></contact></surface></collision>
     </gazebo>
   </xacro:macro>

File: src/perseus_description/urdf/bucket.urdf.xacro (robot description, xacro)
@@ -51,9 +51,15 @@
            L(a)^2 = r^2 + d^2 + 2*r*d*sin(a + lift_phase)
        Retracted (L = 0.365) gives a = -77.61 deg; extended (L = 0.615) gives
-       a = -6.24 deg. So the arms swing 71.36 deg, and at full extension they
-       sit 6.24 deg below the frame's own x axis - they never quite reach
-       horizontal. Joint zero is placed at full extension (top of travel,
-       transport pose) by baking that 6.24 deg into the joint origin, and the
-       joint counts positive DOWN from there: 0 .. 71.36 deg.
+       a = -6.24 deg. So by the CAD the arms swing 71.36 deg, and at full
+       extension they sit 6.24 deg below the frame's own x axis.
+       The real bucket disagrees: at the top of travel its arms are level,
+       parallel to the chassis x axis. So joint zero is the top of travel with
+       the arms LEVEL (lift_zero_pitch is 0), and the joint counts positive
+       DOWN from there. Something in the CAD's lift linkage is therefore 25 mm
+       short - level arms need the rams at 0.640 m pin to pin, not 0.615 - and
+       until that is measured the lift rams are given the stroke the CAD
+       geometry needs for it (lift_ram_stroke). The 71.36 deg of travel is kept
+       as the CAD gives it: on the robot it is the command clamp, so it must
+       not exceed the real travel (TEST.md phase 4 measures it).
        Worth knowing: the CAD's *exported* pose needs L = 0.640, which is 25 mm
        beyond full extension. That is not an error in the CAD - the toolkit
@@ -72,6 +78,14 @@
                             - lift_rod_offset*lift_rod_offset - lift_pivot_drop*lift_pivot_drop)
                            / (2*lift_rod_offset*lift_pivot_drop)}"/>
-  <!-- nose-down pitch of the arm at joint zero, relative to the frame -->
-  <xacro:property name="lift_zero_pitch" value="${-(asin(lift_sin_ext) - lift_phase)}"/>
+  <!-- nose-down pitch of the arm at joint zero, relative to the frame: none,
+       since the real arms are level at the top of travel. The CAD alone would
+       give -(asin(lift_sin_ext) - lift_phase), i.e. 6.24 deg. -->
+  <xacro:property name="lift_zero_pitch" value="0.0"/>
+  <!-- the ram extension that level arms need: L(0) minus the retracted length.
+       0.2748 m, against the 0.250 m stroke of a CAD "250mm Actuator". -->
+  <xacro:property name="lift_ram_stroke"
+                  value="${sqrt(lift_rod_offset*lift_rod_offset + lift_pivot_drop*lift_pivot_drop
+                                + 2*lift_rod_offset*lift_pivot_drop*sin(lift_phase))
+                           - actuator_retracted}"/>
   <xacro:property name="lift_lower" value="0.0"/>
   <!-- 71.36 deg -->
@@ -163,5 +177,5 @@
        meant to hit a ram, and leaving it out keeps contact cheap.
        ═══════════════════════════════════════════════════════════════════ -->
-  <xacro:macro name="bucket_ram" params="name parent mesh xyz mesh_rpy axis phi mesh_xyz:='0 0 0'">
+  <xacro:macro name="bucket_ram" params="name parent mesh xyz mesh_rpy axis phi mesh_xyz:='0 0 0' stroke:=${actuator_stroke}">
     <link name="${prefix}${name}_barrel">
       <inertial>
@@ -201,5 +215,5 @@
       <origin xyz="0 0 0" rpy="0 0 0"/>
       <axis xyz="${axis}"/>
-      <limit lower="0" upper="${actuator_stroke}" effort="50" velocity="0.5"/>
+      <limit lower="0" upper="${stroke}" effort="50" velocity="0.5"/>
       <dynamics damping="0.5"/>
     </joint>
@@ -401,6 +415,6 @@
       </collision>
     </link>
-    <!-- Positive lowers. Zero is the top of travel, with the arms 6.24 deg
-         below the frame axis because that is as far as the actuators reach. -->
+    <!-- Positive lowers. Zero is the top of travel, with the arms level:
+         parallel to the frame and chassis x axis, as on the real bucket. -->
     <joint name="${prefix}bucket_lift_joint" type="revolute">
       <parent link="${prefix}bucket_frame"/>
@@ -591,8 +605,10 @@
     <xacro:bucket_ram name="bucket_ram_lift_left"  parent="bucket_frame" mesh="lift_ram_left"
                       xyz="0.00004 0.099074 -0.24001"
-                      mesh_rpy="0 -1.5707963 -1.5707963" axis="1 0 0" phi="0"/>
+                      mesh_rpy="0 -1.5707963 -1.5707963" axis="1 0 0" phi="0"
+                      stroke="${lift_ram_stroke}"/>
     <xacro:bucket_ram name="bucket_ram_lift_right" parent="bucket_frame" mesh="lift_ram_right"
                       xyz="0.00004 -0.099074 -0.24001"
-                      mesh_rpy="0 -1.5707963 1.5707963" axis="1 0 0" phi="0"/>
+                      mesh_rpy="0 -1.5707963 1.5707963" axis="1 0 0" phi="0"
+                      stroke="${lift_ram_stroke}"/>
     <!-- The tilt ram's barrel is bolted to the plate on the ARMS (the
          tilt_ram_mount pair, via tilt_ram_bracket) and its rod reaches

File: src/perseus_description/urdf/camera_d455_gazebo.xacro (robot description, xacro)
@@ -2,13 +2,29 @@
 <!--
   Gazebo sensors for the RealSense D455.
-  All four are always_on false, so gz renders them only while something is
+  All are always_on false, so gz renders them only while something is
   subscribed - the same pattern the Livox uses in sensors.urdf.xacro. That
-  matters a lot here: with the four sensors rendering unconditionally at 30 Hz,
-  the whole simulation dropped to RTF 0.395 and the Livox fell from 9.8 Hz to
-  3.87 Hz. Rendering is the dominant cost in this world, and only the colour
-  stream has a consumer (vision/aruco_detector, and cube_detector for aligned
-  depth), so paying for infra1/infra2 continuously is pure waste.
-  update_rate is 15 rather than 30 for the same reason. Fiducial acquisition
-  happens while the robot is stationary or turning slowly, so 15 Hz is ample.
+  matters a lot here: with the sensors rendering unconditionally, the whole
+  simulation dropped to RTF 0.395 and the Livox fell from 9.8 Hz to 3.87 Hz.
+  Rendering is the dominant cost in this world, so paying for a stream nobody
+  is subscribed to is pure waste.
+  Resolution and FOV are matched to this robot's actual driver config
+  (sensors/config/realsense.yaml in perseus-v3) rather than picked for sim
+  performance, since vision/stereo_odometry reads camera_info intrinsics and a
+  mismatched FOV or resolution silently changes the scale/geometry it
+  recovers relative to what it'd see on real hardware:
+    - infra1/infra2: 848x480 (depth_module.infra_profile), ~87 deg horizontal
+      FOV (Intel D455 depth-module datasheet spec; not derivable from
+      anything in this repo).
+    - color: 424x240 (rgb_camera.color_profile), ~90 deg horizontal FOV
+      (Intel D455 RGB-module datasheet spec).
+  update_rate is 15 Hz on all four, NOT the real driver's 30 Hz for
+  infra1/infra2, because this sim is rendering-bound: with stereo_odometry
+  subscribed, 848x480 @ 30 Hz alone dragged the sim down to Livox 4.32 Hz
+  (RTF ~0.43) and infra1 itself couldn't even hit its configured 30 Hz,
+  measured at ~13 Hz actual. 15 Hz only affects VO tracking quality (smaller
+  effective baseline motion per matched frame), not the intrinsics/scale
+  correctness the resolution and FOV above are responsible for, so it is the
+  cheaper knob to give up first. Bump back to 30 if this sim ever runs on
+  hardware that can render it without starving Livox.
 -->
 <robot xmlns:xacro="http://ros.org/wiki/xacro">
@@ -41,8 +57,8 @@
         <always_on>false</always_on>
         <camera>
-          <horizontal_fov>1.089</horizontal_fov>
+          <horizontal_fov>1.5708</horizontal_fov>
           <image>
-            <width>640</width>
-            <height>480</height>
+            <width>424</width>
+            <height>240</height>
           </image>
           <clip>
@@ -85,7 +101,7 @@
         <always_on>false</always_on>
         <camera>
-          <horizontal_fov>1.089</horizontal_fov>
+          <horizontal_fov>1.5184</horizontal_fov>
           <image>
-            <width>640</width>
+            <width>848</width>
             <height>480</height>
             <format>L_INT8</format>
@@ -103,5 +119,5 @@
           <visibility_mask>268435454</visibility_mask>
         </camera>
-        <topic>/${name}/${name}/infra1/image_raw</topic>
+        <topic>/${name}/${name}/infra1/image_rect_raw</topic>
         <gz_frame_id>${name}_infra1_optical_frame</gz_frame_id>
       </sensor>
@@ -115,7 +131,7 @@
         <always_on>false</always_on>
         <camera>
-          <horizontal_fov>1.089</horizontal_fov>
+          <horizontal_fov>1.5184</horizontal_fov>
           <image>
-            <width>640</width>
+            <width>848</width>
             <height>480</height>
             <format>L_INT8</format>
@@ -132,6 +148,24 @@
           -->
           <visibility_mask>268435454</visibility_mask>
+          <!--
+            Stereo baseline, in metres, for the Tx term of this camera's own
+            camera_info.P (REP 104: P[3] = -fx * baseline on the right/second camera
+            of a pair; the left camera's Tx conventionally stays 0, so this element
+            is deliberately only on infra2, not infra1). gz::sensors::CameraSensor
+            does NOT derive this from the URDF: there is no code path that measures
+            the actual distance between infra1_frame and infra2_frame and feeds it in.
+            It is a plain SDF field (CameraSensor::Baseline()/SetBaseline()) that
+            defaults to something unrelated to this robot's geometry if left unset.
+            Confirmed live, subscribing to infra2/camera_info's p field: without this
+            element the reported baseline was about 36 mm, not the 95 mm
+            d455_cam_depth_to_infra2_offset actually places the two cameras at, in
+            realsense2_description's own _d455.urdf.xacro. That is silently wrong
+            scale for any stereo algorithm that reads baseline from camera_info
+            rather than from TF, e.g. vision/stereo_odometry's
+            baseline_from_right_projection().
+          -->
+          <baseline>0.095</baseline>
         </camera>
-        <topic>/${name}/${name}/infra2/image_raw</topic>
+        <topic>/${name}/${name}/infra2/image_rect_raw</topic>
         <gz_frame_id>${name}_infra2_optical_frame</gz_frame_id>
       </sensor>

File: src/perseus_description/urdf/perseus.urdf.xacro (robot description, xacro)
@@ -76,5 +76,5 @@
     <link name="${prefix}base_link"/>
     <joint name="${prefix}chassis_joint" type="fixed"> <!-- Joint Connect base_link and chassis -->
-      <origin xyz="${0.2} 0.0 ${chassis_z_offset}" rpy="0.0 0.0 0.0"/>
+      <origin xyz="${0.0} 0.0 ${chassis_z_offset}" rpy="0.0 0.0 0.0"/>
       <parent link="${prefix}base_link"/>
       <child link="${prefix}chassis"/>
