Commit message: Implement per-wheel velocity PID control to mitigate low-speed stalling in the Perseus rover simulation

File: src/perseus/urdf/perseus.urdf.xacro (robot description, xacro)
@@ -4,4 +4,5 @@
   <xacro:arg name="can_bus" default="can0" />
   <xacro:arg name="hardware_plugin" default="perseus_hardware/VescSystemHardware" />
+  <xacro:arg name="use_wheel_pid" default="false" />
   <!-- Import URDF description -->
   <xacro:include filename="$(find perseus_description)/urdf/perseus.urdf.xacro" />
@@ -12,4 +13,4 @@
   <!-- Instantiate the description and the ROS2 control information -->
   <xacro:perseus prefix="$(arg prefix)" />
-  <xacro:perseus_ros2_control name="Perseus" prefix="$(arg prefix)" can_bus="$(arg can_bus)" hardware_plugin="$(arg hardware_plugin)"/>
+  <xacro:perseus_ros2_control name="Perseus" prefix="$(arg prefix)" can_bus="$(arg can_bus)" hardware_plugin="$(arg hardware_plugin)" use_wheel_pid="$(arg use_wheel_pid)"/>
 </robot>

File: src/perseus_description/ros2_control/perseus.ros2_control.xacro (robot description, xacro)
@@ -1,5 +1,5 @@
 <?xml version="1.0"?>
 <robot xmlns:xacro="http://www.ros.org/wiki/xacro">
-  <xacro:macro name="perseus_ros2_control" params="namespace:='' name prefix can_bus:='can0' hardware_plugin">
+  <xacro:macro name="perseus_ros2_control" params="namespace:='' name prefix can_bus:='can0' hardware_plugin use_wheel_pid:='false'">
     <ros2_control name="${name}" type="system">
       <hardware>
@@ -34,4 +34,14 @@
           </ros>
           <parameters>$(find perseus)/config/perseus_controllers.yaml</parameters>
+          <!-- Overlay, so it MUST come after the base file for its overrides to
+               win. This is the sim equivalent of the second parameter file
+               controllers.launch.py passes on the rover. -->
+          <!-- Used bare, not compared against a string: xacro has already
+               coerced "true" into a Python bool by this point, so
+               ${use_wheel_pid == 'true'} silently evaluates False (it compares a
+               bool to a string). Bare, it handles true/false/True/1/0 alike. -->
+          <xacro:if value="${use_wheel_pid}">
+            <parameters>$(find perseus)/config/wheel_pid_chaining.yaml</parameters>
+          </xacro:if>
           <parameters>$(find perseus_simulation)/config/ros2_control_sim.yaml</parameters>
         </plugin>

Commit message: Replace the bucket model with perseus-v3's mount and pivots
Reverts the Onshape-derived bucket (033efe5, bb1a12f) and ports the
implementation from perseus-v3 in its place, so the simulation and the rover
describe the same attachment.

What perseus-v3 models is the mount itself, not the linkage: a bucket_mount
link carrying bucket_mount.dae, plus the four lift-arm pivots as bare frames
at the centres of the bearing blocks moulded into that mesh. Five links, no
joints to drive. bucket.urdf.xacro is byte-identical to perseus-v3's apart
from the package name in the mesh path.

The reverted model had two actuated DOFs and three rams, which is why
everything built around them goes with it: bucket_ram_follower.py (it solved
the ram angles in closed form because dartsim refuses closed loops), the
/bucket/* bridge topics those controllers consumed, the 22 STLs, the Onshape
export under cad/bucket, and docs/bucket-{urdf,changelog}.md. None of it has
anything to attach to now. Recoverable from the reverted commits if the
articulated model is wanted again.

Also swaps the use_bucket flag for perseus-v3's payload argument, which this
repo already declared for the driver node but not for the description, so one
argument now selects both. payload:=bucket is threaded through
robot_state_publisher.launch.py, and view_perseus.launch.py gains the argument
so the mount can be viewed in RViz without Gazebo. perseus_sim.launch.py
defaults it to bucket, matching what use_bucket did there.

Verified with pixi run build: the xacro expands to 34 links at payload:=none
and 39 at payload:=bucket, the five added being bucket_mount and the four
bucket_lift_arm_pivot_* frames.

File: src/perseus/urdf/perseus.urdf.xacro (robot description, xacro)
@@ -4,6 +4,5 @@
   <xacro:arg name="can_bus" default="can0" />
   <xacro:arg name="hardware_plugin" default="perseus_hardware/VescSystemHardware" />
-  <!-- Attach the excavation bucket. Off by default; perseus_sim.launch.py turns it on. -->
-  <xacro:arg name="use_bucket" default="false" />
+  <xacro:arg name="payload" default="none" />
   <!-- Import URDF description -->
   <xacro:include filename="$(find perseus_description)/urdf/perseus.urdf.xacro" />
@@ -13,5 +12,5 @@
   <xacro:include filename="$(find perseus_description)/ros2_control/perseus.ros2_control.xacro" />
   <!-- Instantiate the description and the ROS2 control information -->
-  <xacro:perseus prefix="$(arg prefix)" />
+  <xacro:perseus prefix="$(arg prefix)" payload="$(arg payload)" />
   <xacro:perseus_ros2_control name="Perseus" prefix="$(arg prefix)" can_bus="$(arg can_bus)" hardware_plugin="$(arg hardware_plugin)"/>
 </robot>
