Commit message: Replace the bucket model with perseus-v3's mount and pivots
Reverts the Onshape-derived bucket (033efe5, bb1a12f) and ports the
implementation from perseus-v3 in its place, so the simulation and the rover
describe the same attachment.

What perseus-v3 models is the mount itself, not the linkage: a bucket_mount
link carrying bucket_mount.dae, plus the four lift-arm pivots as bare frames
at the centres of the bearing blocks moulded into that mesh. Five links, no
joints to drive. bucket.urdf.xacro is byte-identical to perseus-v3's apart
from the package name in the mesh path.

The reverted model had two actuated DOFs and three rams, which is why
everything built around them goes with it: bucket_ram_follower.py (it solved
the ram angles in closed form because dartsim refuses closed loops), the
/bucket/* bridge topics those controllers consumed, the 22 STLs, the Onshape
export under cad/bucket, and docs/bucket-{urdf,changelog}.md. None of it has
anything to attach to now. Recoverable from the reverted commits if the
articulated model is wanted again.

Also swaps the use_bucket flag for perseus-v3's payload argument, which this
repo already declared for the driver node but not for the description, so one
argument now selects both. payload:=bucket is threaded through
robot_state_publisher.launch.py, and view_perseus.launch.py gains the argument
so the mount can be viewed in RViz without Gazebo. perseus_sim.launch.py
defaults it to bucket, matching what use_bucket did there.

Verified with pixi run build: the xacro expands to 34 links at payload:=none
and 39 at payload:=bucket, the five added being bucket_mount and the four
bucket_lift_arm_pivot_* frames.

File: src/perseus_description/urdf/perseus.urdf.xacro (robot description, xacro)
@@ -1,5 +1,5 @@
 <?xml version="1.0"?>
 <robot xmlns:xacro="http://ros.org/wiki/xacro">
-  <xacro:macro name="perseus" params="prefix">
+  <xacro:macro name="perseus" params="prefix payload:=none">
     <!-- Motors Properties -->
     <xacro:property name="motors_y_offset" value="0.035"/>
@@ -69,6 +69,6 @@
     <xacro:include filename="$(find perseus_description)/urdf/sensors.urdf.xacro"/>
     <xacro:include filename="$(find perseus_description)/urdf/sensor_mount.urdf.xacro"/>
+    <xacro:include filename="$(find perseus_description)/urdf/bucket.urdf.xacro"/>
     <xacro:include filename="$(find perseus_description)/urdf/camera_d455_gazebo.xacro"/>
-    <xacro:include filename="$(find perseus_description)/urdf/bucket.urdf.xacro"/>
     <xacro:include filename="$(find realsense2_description)/urdf/_d455.urdf.xacro"/>
     <!-- An empty base_link to attach everything to -->
@@ -95,12 +95,7 @@
     <!-- Livox and RealSense both hang off the mast: see sensor_mount.urdf.xacro -->
     <xacro:sensor_mount prefix="${prefix}"/>
-    <!--
-      Excavation bucket, bolted to the front face of the chassis. Off by
-      default so every existing launch keeps the bare rover; the simulation
-      turns it on. See bucket.urdf.xacro for the geometry and for how the
-      four-bar linkage is reduced to its two driven joints.
-    -->
-    <xacro:if value="$(arg use_bucket)">
-      <xacro:bucket parent="${prefix}chassis"/>
+    <!-- payload:=bucket attaches the bucket mount to the chassis; see bucket.urdf.xacro -->
+    <xacro:if value="${payload == 'bucket'}">
+      <xacro:bucket prefix="${prefix}"/>
     </xacro:if>
   </xacro:macro>

Commit message: Port perseus-v3's bucket linkage and its ros2_control controllers
Replaces the mount-only bucket from fe29ecd with perseus-v3's current
description: the mount plus the lift arms, bucket, jaw, five rams and encoder
frames. bucket.urdf.xacro is v3's file with only the mesh path changed; the 33
meshes move under meshes/bucket/ as in v3, so the old top-level
bucket_mount.dae goes.

The Gazebo-only parts live in bucket.gazebo.xacro so the description stays a
straight copy: position controllers for the ten ram joints, a joint state
publisher for them, and the contact friction. The rams are driven by v3's
bucket_ram_follower.py, now in perseus_description as in v3, which perseus_sim
runs for payload:=bucket and view_perseus runs in viewer mode.

lift, tilt and jaw are ros2_control joints (bucket.ros2_control.xacro, on
GazeboSimSystem in the sim), driven by the controllers from v3's
payloads/config/bucket_controller.yaml (bucket_controllers.yaml here). The
bucket_controller launch argument takes the same choices and default as v3's
perseus.launch.py. The bucket shares the drive's controller_manager, because
gz_ros2_control runs one per model, but its controller is spawned into the
payloads namespace, so goals go to the same action as on the robot:
/payloads/<controller>/follow_joint_trajectory. Adds
joint_trajectory_controller to pixi.toml.

v3's linkage meshes segfaulted the Gazebo server in gz-common's Collada
polylist loader. They are Assimp exports whose VERTEX and NORMAL inputs share
offset 0; RViz reads that, gz-common does not. Each now gives NORMAL its own
offset with the index list interleaved to match; the geometry is unchanged.

Verified in the arena world: all three controllers activate, a
FollowJointTrajectory goal of lift 45, tilt -15, jaw 30 deg returns SUCCEEDED
with every joint on target, the rams track, and TF resolves base_link to
bucket_jaw.

File: src/perseus/urdf/perseus.urdf.xacro (robot description, xacro)
@@ -14,3 +14,7 @@
   <xacro:perseus prefix="$(arg prefix)" payload="$(arg payload)" />
   <xacro:perseus_ros2_control name="Perseus" prefix="$(arg prefix)" can_bus="$(arg can_bus)" hardware_plugin="$(arg hardware_plugin)"/>
+  <xacro:if value="${'$(arg payload)' == 'bucket'}">
+    <xacro:include filename="$(find perseus_description)/ros2_control/bucket.ros2_control.xacro" />
+    <xacro:bucket_ros2_control prefix="$(arg prefix)" hardware_plugin="$(arg hardware_plugin)"/>
+  </xacro:if>
 </robot>

File: src/perseus_description/ros2_control/perseus.ros2_control.xacro (robot description, xacro)
@@ -34,4 +34,5 @@
           </ros>
           <parameters>$(find perseus)/config/perseus_controllers.yaml</parameters>
+          <parameters>$(find perseus_simulation)/config/bucket_controllers.yaml</parameters>
           <parameters>$(find perseus_simulation)/config/ros2_control_sim.yaml</parameters>
         </plugin>
