Commit message: Port perseus-v3's bucket linkage and its ros2_control controllers
Replaces the mount-only bucket from fe29ecd with perseus-v3's current
description: the mount plus the lift arms, bucket, jaw, five rams and encoder
frames. bucket.urdf.xacro is v3's file with only the mesh path changed; the 33
meshes move under meshes/bucket/ as in v3, so the old top-level
bucket_mount.dae goes.

The Gazebo-only parts live in bucket.gazebo.xacro so the description stays a
straight copy: position controllers for the ten ram joints, a joint state
publisher for them, and the contact friction. The rams are driven by v3's
bucket_ram_follower.py, now in perseus_description as in v3, which perseus_sim
runs for payload:=bucket and view_perseus runs in viewer mode.

lift, tilt and jaw are ros2_control joints (bucket.ros2_control.xacro, on
GazeboSimSystem in the sim), driven by the controllers from v3's
payloads/config/bucket_controller.yaml (bucket_controllers.yaml here). The
bucket_controller launch argument takes the same choices and default as v3's
perseus.launch.py. The bucket shares the drive's controller_manager, because
gz_ros2_control runs one per model, but its controller is spawned into the
payloads namespace, so goals go to the same action as on the robot:
/payloads/<controller>/follow_joint_trajectory. Adds
joint_trajectory_controller to pixi.toml.

v3's linkage meshes segfaulted the Gazebo server in gz-common's Collada
polylist loader. They are Assimp exports whose VERTEX and NORMAL inputs share
offset 0; RViz reads that, gz-common does not. Each now gives NORMAL its own
offset with the index list interleaved to match; the geometry is unchanged.

Verified in the arena world: all three controllers activate, a
FollowJointTrajectory goal of lift 45, tilt -15, jaw 30 deg returns SUCCEEDED
with every joint on target, the rams track, and TF resolves base_link to
bucket_jaw.

File: src/perseus_description/urdf/bucket.urdf.xacro (robot description, xacro)
@@ -1,4 +1,636 @@
 <?xml version="1.0"?>
 <robot name="bucket" xmlns:xacro="http://ros.org/wiki/xacro">
+  <!-- Arm-pivot midpoint relative to bucket_mount's origin, the centre of the frame's
+       front face (frame-mesh coordinates: face centre (0.0174, 0.4607, 0.093), pivot
+       midpoint (0.0591, 0.44071, 0.213)). x and z agree with the +0.042 / +-0.12 that
+       bucket.urdf.xacro puts its lift pivot frames at.
+       y is 0: bucket_frame, bucket_lift_arm, bucket_body and bucket_jaw all sit on the
+       machine centre line, like bucket_mount, so a frame's y tells you how far off
+       centre a part is rather than where the CAD happened to put its origin. The CAD is
+       offset - its arm pivots are at -0.12 and +0.08 from the face centre, and the
+       bucket hangs off one arm - and that offset now lives in the child origins inside
+       each link instead of in the frame itself. Nothing moves: lift, tilt and jaw all
+       turn about y, so sliding a frame along y leaves its axis line exactly where it
+       was, at any joint angle. -->
+  <xacro:property name="bucket_frame_x" value="0.0417"/>
+  <xacro:property name="bucket_frame_y" value="0.0"/>
+  <xacro:property name="bucket_frame_z" value="0.120"/>
+  <!-- ══ Density ═════════════════════════════════════════════════════════
+       The ONE genuine assumption in this file. Onshape reports
+       "hasMass": false, "massMissingCount": 53 for this assembly - not a
+       single part has a material assigned, which is why the export wrote
+       mass=0 or mass=1 everywhere. The *volumes* are exact though (Onshape
+       gives 4138.7 cm3 for the assembly; summing the meshes here gives
+       4118.4 cm3, a 0.5% tessellation difference), so mass is volume x this.
+       2700 kg/m3 is 6061 aluminium. The frame and rails measure 20x20 mm
+       V-slot extrusion at ~70% fill, and the parts list contains a
+       "BucketClipVslotMount", so extruded aluminium is the right call. For a
+       steel fabrication use 7850 and every mass and inertia below scales by
+       2.907 - they are all linear in density.
+       To fix this properly: assign materials to every part in Onshape and
+       re-export. Nothing else will. -->
+  <xacro:property name="bucket_density" value="2700.0"/>
+  <!-- ══ Linkage geometry ════════════════════════════════════════════════
+       All MEASURED, by forward-kinematicking the export's mate transforms
+       into one frame. Mate transforms are rigid-body facts and are unaffected
+       by the export's broken mass properties. -->
+  <!-- arm pivot -> bucket pivot, along the arm -->
+  <xacro:property name="arm_length" value="0.70004"/>
+  <!-- arm pivot -> lift-actuator bracket, along the arm (Fastened_2) -->
+  <xacro:property name="lift_rod_offset" value="0.59712"/>
+  <!-- arm pivot above the lift-actuator pivot -->
+  <xacro:property name="lift_pivot_drop" value="0.24000"/>
+  <!-- the lift bracket sits this far below the pivot line, hence the phase -->
+  <xacro:property name="lift_phase" value="-0.016763"/>   <!-- -0.96 deg -->
+  <!-- pin-to-pin length of a "250mm Actuator" as drawn in CAD = retracted -->
+  <xacro:property name="actuator_retracted" value="0.36500"/>
+  <xacro:property name="actuator_stroke" value="0.25000"/>
+  <!-- ══ Lift travel ═════════════════════════════════════════════════════
+       DERIVED from the above. With r the bracket radius, d the pivot drop and
+       a the arm angle measured from the CAD pose,
+           L(a)^2 = r^2 + d^2 + 2*r*d*sin(a + lift_phase)
+       Retracted (L = 0.365) gives a = -77.61 deg; extended (L = 0.615) gives
+       a = -6.24 deg. So the arms swing 71.36 deg, and at full extension they
+       sit 6.24 deg below the frame's own x axis - they never quite reach
+       horizontal. Joint zero is placed at full extension (top of travel,
+       transport pose) by baking that 6.24 deg into the joint origin, and the
+       joint counts positive DOWN from there: 0 .. 71.36 deg.
+       Worth knowing: the CAD's *exported* pose needs L = 0.640, which is 25 mm
+       beyond full extension. That is not an error in the CAD - the toolkit
+       places each link by its own mate transform and never solves the loop, so
+       the exported pose is the mate zero, not an assembly configuration. It is
+       also why the pose in cad/bucket/ has the actuators visibly detached from
+       their brackets. -->
+  <xacro:property name="lift_len_max"
+                  value="${sqrt(lift_rod_offset*lift_rod_offset + lift_pivot_drop*lift_pivot_drop)}"/>
+  <xacro:property name="lift_sin_ext"
+                  value="${((actuator_retracted + actuator_stroke)**2
+                            - lift_rod_offset*lift_rod_offset - lift_pivot_drop*lift_pivot_drop)
+                           / (2*lift_rod_offset*lift_pivot_drop)}"/>
+  <xacro:property name="lift_sin_ret"
+                  value="${(actuator_retracted**2
+                            - lift_rod_offset*lift_rod_offset - lift_pivot_drop*lift_pivot_drop)
+                           / (2*lift_rod_offset*lift_pivot_drop)}"/>
+  <!-- nose-down pitch of the arm at joint zero, relative to the frame -->
+  <xacro:property name="lift_zero_pitch" value="${-(asin(lift_sin_ext) - lift_phase)}"/>
+  <xacro:property name="lift_lower" value="0.0"/>
+  <!-- 71.36 deg -->
+  <xacro:property name="lift_upper" value="${asin(lift_sin_ext) - asin(lift_sin_ret)}"/>
+  <!-- ══ Tilt travel ═════════════════════════════════════════════════════
+       Same treatment. The tilt actuator works between a pin on the bucket
+       131.1 mm from the bucket pivot and a bracket on the arm 513.5 mm from
+       it. The included angle is 108.25 deg in the CAD pose. Extending to
+       0.615 m opens it to 136.34 deg (the bucket dumps); retracting closes it,
+       but the actuator's 0.365 m retracted length is unreachable - the two
+       pins go collinear at 0.382 m first, so the geometric stop is the fold at
+       0 deg, i.e. 1.889 rad of curl.
+       Curl is capped short of that fold: past about 1.6 rad the bucket is
+       folded back over the arms, which the real structure will not allow.
+       Dump is the true actuator limit.
+       The joint counts positive toward DUMP (tipping down) from the CAD pose,
+       so curl is negative: -91.673 (curl) .. +28.098 (dump) deg. -->
+  <xacro:property name="tilt_lower" value="${radians(-91.673)}"/>
+  <xacro:property name="tilt_upper" value="${radians(28.098)}"/>
+  <!-- geometric, for reference -->
+  <xacro:property name="tilt_fold_limit" value="1.889229"/>
+  <!-- ══ Actuator force and speed ════════════════════════════════════════
+       0.1 m/s is ACTUATOR_MAX_SPEED from bucket_driver.cpp in the `payloads`
+       package - the real robot's own number. Force is a 1.5 kN class 250 mm
+       actuator through the measured moment arms: 224 mm at the lift pivot,
+       113 mm at the tilt pivot. For scale, holding the arm and a full bucket
+       out straight takes about 41 Nm. -->
+  <xacro:property name="lift_moment_arm" value="0.2239"/>
+  <xacro:property name="tilt_moment_arm" value="0.1126"/>
+  <xacro:property name="actuator_force" value="1500.0"/>
+  <xacro:property name="actuator_speed" value="0.1"/>
+  <xacro:property name="lift_effort" value="${actuator_force*lift_moment_arm}"/>
+  <xacro:property name="tilt_effort" value="${actuator_force*tilt_moment_arm}"/>
+  <xacro:property name="lift_velocity" value="${actuator_speed/lift_moment_arm}"/>
+  <xacro:property name="tilt_velocity" value="${actuator_speed/tilt_moment_arm}"/>
+  <!-- ══ Jaw travel ══════════════════════════════════════════════════════
+       Same treatment as lift and tilt. The FRONT half hinges at the plate
+       apexes and the 50 mm actuator's rod pin sits only 63 mm from the hinge,
+       with the base pin 202 mm below it. A stroke of 50 mm therefore sweeps
+       0.84 rad (48 deg), and dL/dtheta at the CAD pose is 0.0615 m/rad - that
+       is the moment arm below. The actuators are planar (see "Jaw rams"), so
+       the length is just the in-plane pin-to-pin distance, 0.2068 m extended.
+       Which end of the stroke is the CAD pose? Neither the export nor the mate
+       limits say (the toolkit fills every slider with a default -0.25..0), so
+       this was confirmed against the real machine: the CAD is drawn with the
+       actuators fully EXTENDED - the FRONT frame is already tight against the
+       REAR frame and cannot be pushed any closer - so the jaws can only open
+       from there:
+           extended end (CAD pose) : theta =  0.0000
+           retracted end           : theta = -0.8376   (L falls by 50 mm)
+       (The other reading would give 0 .. +1.0540; it does not apply.)
+       The joint is -theta, so it counts positive OPENING from closed:
+       0 .. 47.991 deg. -->
+  <xacro:property name="jaw_lower" value="0.0"/>
+  <xacro:property name="jaw_upper" value="${radians(47.991)}"/>
+  <xacro:property name="jaw_moment_arm" value="0.0615"/>
+  <xacro:property name="jaw_effort" value="${actuator_force*jaw_moment_arm}"/>
+  <xacro:property name="jaw_velocity" value="${actuator_speed/jaw_moment_arm}"/>
+  <!-- ══ Masses: exact CAD volume x density ══════════════════════════════ -->
+  <xacro:property name="v_frame" value="0.00051813"/>   <!-- Frame_Repaired_1     -->
+  <xacro:property name="v_plate" value="0.00015904"/>   <!-- one bearing block    -->
+  <xacro:property name="v_tube" value="0.00016847"/>    <!-- one arm, 40x20x2 tube-->
+  <xacro:property name="v_bracket" value="0.00001293"/> <!-- one actuator bracket -->
+  <xacro:property name="v_arm_mount" value="0.00003805"/><!-- one on-arm plate    -->
+  <xacro:property name="v_actuator" value="0.00040493"/><!-- one 250 mm actuator  -->
+  <!-- the whole clamshell -->
+  <xacro:property name="v_bucket" value="0.00129748"/>
+  <xacro:property name="m_frame" value="${v_frame*bucket_density}"/>
+  <xacro:property name="m_plate" value="${v_plate*bucket_density}"/>
+  <xacro:property name="m_tube" value="${v_tube*bucket_density}"/>
+  <xacro:property name="m_bracket" value="${v_bracket*bucket_density}"/>
+  <xacro:property name="m_arm_mount" value="${v_arm_mount*bucket_density}"/>
+  <xacro:property name="m_half_act" value="${v_actuator*bucket_density/2}"/>
+  <xacro:property name="m_bucket" value="${v_bucket*bucket_density}"/>
+  <!-- Body totals and their inertia tensors were composed from the meshes
+       (exact tetrahedron integration, then parallel axis) plus the lumped
+       actuator halves. At 2700 kg/m3 they come to 4.210 / 2.860 / 4.050 kg.
+       Both mass and inertia are linear in density, so the scale factor below
+       keeps the whole file correct if you change bucket_density. -->
+  <xacro:property name="k" value="${bucket_density/2700.0}"/>
+  <xacro:property name="M" value="file://$(find perseus_description)/meshes/bucket"/>
+  <!-- ══ Rams ════════════════════════════════════════════════════════════
+       One ram = barrel (revolute on its parent) + shaft (prismatic on the
+       barrel). `phi` rotates the joint zero so the travel range does not
+       straddle +/-pi; the follower node publishes beta + phi.
+       Mass is a token 20 g: the real 1.09 kg per ram is already lumped at the
+       pin locations on the frame, arm and bucket, and double-counting it here
+       would change the linkage dynamics. No collision geometry - nothing is
+       meant to hit a ram, and leaving it out keeps contact cheap.
+       ═══════════════════════════════════════════════════════════════════ -->
+  <xacro:macro name="bucket_ram" params="name parent mesh xyz mesh_rpy axis phi mesh_xyz:='0 0 0'">
+    <link name="${prefix}${name}_barrel">
+      <inertial>
+        <origin xyz="0.15 0 0" rpy="0 0 0"/>
+        <mass value="0.02"/>
+        <xacro:box_inertia m="0.02" x="0.34" y="0.06" z="0.06"/>
+      </inertial>
+      <visual>
+        <origin xyz="${mesh_xyz}" rpy="${mesh_rpy}"/>
+        <geometry><mesh scale="1.0 1.0 1.0" filename="${M}/${mesh}_barrel.dae"/></geometry>
+        <material name="bucket_steel"/>
+      </visual>
+    </link>
+    <joint name="${prefix}${name}_pitch_joint" type="revolute">
+      <parent link="${prefix}${parent}"/>
+      <child link="${prefix}${name}_barrel"/>
+      <origin xyz="${xyz}" rpy="0 ${phi} 0"/>
+      <axis xyz="0 -1 0"/>
+      <limit lower="-1.8" upper="1.8" effort="50" velocity="5"/>
+      <dynamics damping="0.5"/>
+    </joint>
+    <link name="${prefix}${name}_shaft">
+      <inertial>
+        <origin xyz="0.25 0 0" rpy="0 0 0"/>
+        <mass value="0.02"/>
+        <xacro:box_inertia m="0.02" x="0.29" y="0.02" z="0.02"/>
+      </inertial>
+      <visual>
+        <origin xyz="${mesh_xyz}" rpy="${mesh_rpy}"/>
+        <geometry><mesh scale="1.0 1.0 1.0" filename="${M}/${mesh}_shaft.dae"/></geometry>
+        <material name="bucket_dark"/>
+      </visual>
+    </link>
+    <joint name="${prefix}${name}_extend_joint" type="prismatic">
+      <parent link="${prefix}${name}_barrel"/>
+      <child link="${prefix}${name}_shaft"/>
+      <origin xyz="0 0 0" rpy="0 0 0"/>
+      <axis xyz="${axis}"/>
+      <limit lower="0" upper="${actuator_stroke}" effort="50" velocity="0.5"/>
+      <dynamics damping="0.5"/>
+    </joint>
+    <!-- Cosmetic: no gravity, so they hold their pose if the follower node is
+         not running rather than collapsing. -->
+    <gazebo reference="${prefix}${name}_barrel"><gravity>false</gravity></gazebo>
+    <gazebo reference="${prefix}${name}_shaft"><gravity>false</gravity></gazebo>
+  </xacro:macro>
+  <!-- ══ Jaw rams ════════════════════════════════════════════════════════
+       The two 50 mm jaw actuators, animated. Each is a barrel pinned to the REAR
+       half by a pitch joint plus a rod on a prismatic joint, exactly like the
+       250 mm rams above, and both sides share one angle and one extension.
+       They are PLANAR. The pin positions read straight off the CAD mates are the
+       mate-connector origins, which sit on each pin line but not at its centre:
+       the barrel's is 22.9 mm / -9.2 mm off along the pin axis and the rod's is
+       20.1 mm. Correcting for that puts the barrel pin and the rod pin of each
+       actuator in the same plane (y = -0.0814 and +0.3254), so there is no
+       sideways skew and pitch alone aims the barrel. (An earlier version of these
+       notes claimed a 27 mm skew needing a 3-D follower; that was the connector
+       offset, not a real skew.)
+       Joint zero is the CAD pose, with the actuators fully extended, so the model
+       is right in RViz without the follower running. ext runs 0 (extended) down to
+       -0.05 (retracted). Mass is a token 20 g: the real masses are already in the
+       REAR and jaw links, and there is no collision. -->
+  <xacro:property name="jaw_ram_x" value="0.00974"/>
+  <xacro:property name="jaw_ram_z" value="-0.03206"/>
+  <xacro:property name="jaw_ram_phi0" value="-1.54342"/>
+  <xacro:property name="jaw_ram_len" value="0.20681"/>
+  <xacro:property name="jaw_ram_stroke" value="0.05"/>
+  <xacro:macro name="bucket_jaw_ram" params="name y base_mesh shaft_mesh barrel_xyz barrel_rpy shaft_xyz shaft_rpy">
+    <link name="${prefix}${name}_barrel">
+      <inertial>
+        <origin xyz="0.07 0 0" rpy="0 0 0"/>
+        <mass value="0.02"/>
+        <xacro:box_inertia m="0.02" x="0.15" y="0.04" z="0.04"/>
+      </inertial>
+      <visual>
+        <origin xyz="${barrel_xyz}" rpy="${barrel_rpy}"/>
+        <geometry><mesh scale="1.0 1.0 1.0" filename="${M}/${base_mesh}.dae"/></geometry>
+        <material name="bucket_dark"/>
+      </visual>
+    </link>
+    <joint name="${prefix}${name}_pitch_joint" type="revolute">
+      <parent link="${prefix}bucket_body"/>
+      <child link="${prefix}${name}_barrel"/>
+      <origin xyz="${jaw_ram_x} ${y} ${jaw_ram_z}" rpy="0 ${jaw_ram_phi0} 0"/>
+      <axis xyz="0 1 0"/>
+      <limit lower="-0.6" upper="0.6" effort="20" velocity="5"/>
+      <dynamics damping="0.005"/>
+    </joint>
+    <link name="${prefix}${name}_shaft">
+      <inertial>
+        <origin xyz="0.14 0 0" rpy="0 0 0"/>
+        <mass value="0.02"/>
+        <xacro:box_inertia m="0.02" x="0.09" y="0.02" z="0.02"/>
+      </inertial>
+      <visual>
+        <origin xyz="${shaft_xyz}" rpy="${shaft_rpy}"/>
+        <geometry><mesh scale="1.0 1.0 1.0" filename="${M}/${shaft_mesh}.dae"/></geometry>
+        <material name="bucket_steel"/>
+      </visual>
+    </link>
+    <joint name="${prefix}${name}_extend_joint" type="prismatic">
+      <parent link="${prefix}${name}_barrel"/>
+      <child link="${prefix}${name}_shaft"/>
+      <origin xyz="0 0 0" rpy="0 0 0"/>
+      <axis xyz="1 0 0"/>
+      <limit lower="${-jaw_ram_stroke}" upper="0" effort="20" velocity="0.5"/>
+      <dynamics damping="0.3"/>
+    </joint>
+    <gazebo reference="${prefix}${name}_barrel"><gravity>false</gravity></gazebo>
+    <gazebo reference="${prefix}${name}_shaft"><gravity>false</gravity></gazebo>
+  </xacro:macro>
+  <!-- ══ Encoder frames ══════════════════════════════════════════════════
+       bucket_driver reads LIFT_BOTH / TILT_BOTH / JAWS_BOTH: one encoder at each
+       END of each pivot axis, six in all. The URDF has one joint per axis, which
+       sits at a single point along it, so the other end had no frame at all. These
+       are plain fixed frames on the FIXED side of each joint, exactly on its axis
+       at the circled bearing blocks / plate apexes, so both ends of every axis are
+       visible and each frame takes the joint's axis orientation. "left" is +y.
+       They carry no mass or geometry, so they change nothing physically. -->
+  <xacro:macro name="bucket_encoder" params="name parent xyz">
+    <link name="${prefix}${name}"/>
+    <joint name="${prefix}${name}_joint" type="fixed">
+      <parent link="${prefix}${parent}"/>
+      <child link="${prefix}${name}"/>
+      <origin xyz="${xyz}" rpy="0 0 0"/>
+    </joint>
+  </xacro:macro>
+  <xacro:macro name="bucket_linkage" params="prefix:=^">
+    <!--
+      The moving parts of the excavation bucket: lift arms, bucket, clamshell jaw, the
+      five actuator rams and the six encoder frames. They hang off the `bucket_mount`
+      link that the `bucket` macro below defines, at the arm-pivot midpoint; the frame
+      body itself is drawn there by bucket_mount.dae, not here.
+      Derived from the perseus_simulation `bucket-urdf` branch's bucket.urdf.xacro,
+      which holds the full derivation (CAD dimensions, joint limits, masses, the
+      closed-form ram kinematics) in its header and in docs/bucket-urdf.md there. Two
+      deliberate differences:
+        * the frame link is kept only as an inertial (its mass and inertia, no
+          visual), because bucket_mount.dae already draws the frame;
+        * the <gazebo> blocks (joint position controllers, joint state publisher) are
+          left out - this repo does not simulate the bucket.
+      Joints: bucket_lift_joint, bucket_tilt_joint and bucket_jaw_joint are the three
+      driven ones, matching bucket_driver's LIFT_BOTH / TILT_BOTH / JAWS_BOTH. The ten
+      ram joints (five rams, each a pitch and an extend) are not free: they are
+      functions of those three and are set by scripts/bucket_ram_follower.py, which
+      view_perseus.launch.py starts for payload:=bucket. Nothing else drives them, so
+      without it the rams sit at their zero pose.
+      This block and the materials below live inside the macro, not at file top level,
+      so payload:=none carries none of it - not even as a comment.
+    -->
+    <!-- Materials, likewise kept inside the macro. -->
+    <material name="bucket_arm_blue">
+      <color rgba="0.13 0.25 0.50 1.0"/>
+    </material>
+    <material name="bucket_dark">
+      <color rgba="0.20 0.22 0.25 1.0"/>
+    </material>
+    <material name="bucket_steel">
+      <color rgba="0.55 0.60 0.65 1.0"/>
+    </material>
+    <!-- Sits at the arm-pivot midpoint with base_link axes. Inertial only: the frame
+         is drawn by bucket_mount. Mass is the frame plus half of each lift ram. -->
+    <link name="${prefix}bucket_frame">
+      <inertial>
+        <origin xyz="-0.033899 -0.000002 -0.155044" rpy="0 0 0"/>
+        <mass value="${4.2099*k}"/>
+        <inertia ixx="${0.114994*k}" ixy="${0.0*k}"      ixz="${0.001957*k}"
+                                     iyy="${0.060850*k}" iyz="${0.0*k}"
+                                                         izz="${0.072903*k}"/>
+      </inertial>
+    </link>
+    <joint name="${prefix}bucket_frame_joint" type="fixed">
+      <parent link="${prefix}bucket_mount"/>
+      <child link="${prefix}bucket_frame"/>
+      <origin xyz="${bucket_frame_x} ${bucket_frame_y} ${bucket_frame_z}" rpy="0 0 0"/>
+    </joint>
+    <!-- ═══════════════════════════════════════════════════════════════════
+         Arms: both tubes, both lift brackets, the tilt-actuator plate and its
+         bracket, as one rigid body - the bucket pins them together at the far
+         end so they cannot move relative to each other.
+         Both tubes are the same part ("Left Arm - Square Tube" <1> and <2>);
+         there is no right-hand mirror in the CAD, so both are offset the same
+         way from their pivots rather than symmetrically. That is reproduced
+         faithfully here.
+         ═══════════════════════════════════════════════════════════════════ -->
+    <link name="${prefix}bucket_lift_arm">
+      <inertial>
+        <origin xyz="0.407179 -0.000305 -0.000497" rpy="0 0 0"/>
+        <mass value="${2.8599*k}"/>
+        <inertia ixx="${0.022280*k}" ixy="${0.000424*k}" ixz="${0.004437*k}"
+                                     iyy="${0.125578*k}" iyz="${0.000055*k}"
+                                                         izz="${0.147197*k}"/>
+      </inertial>
+      <visual>
+        <origin xyz="0.00004 0.08 -0.00001" rpy="1.5707963 0 0"/>
+        <geometry><mesh scale="1.0 1.0 1.0" filename="${M}/lift_arm_left.dae"/></geometry>
+        <material name="bucket_arm_blue"/>
+      </visual>
+      <visual>
+        <origin xyz="0.00004 -0.12 -0.00001" rpy="1.5707963 0 0"/>
+        <geometry><mesh scale="1.0 1.0 1.0" filename="${M}/lift_arm_right.dae"/></geometry>
+        <material name="bucket_arm_blue"/>
+      </visual>
+      <visual>
+        <origin xyz="0.59704 -0.1 -0.01001" rpy="0 0 -1.5707963"/>
+        <geometry><mesh scale="1.0 1.0 1.0" filename="${M}/lift_ram_bracket_right.dae"/></geometry>
+        <material name="bucket_dark"/>
+      </visual>
+      <visual>
+        <origin xyz="0.59704 0.1 -0.01001" rpy="0 0 -1.5707963"/>
+        <geometry><mesh scale="1.0 1.0 1.0" filename="${M}/lift_ram_bracket_left.dae"/></geometry>
+        <material name="bucket_dark"/>
+      </visual>
+      <visual>
+        <origin xyz="0.22674 -0.1 0.00999" rpy="3.1415927 0 0"/>
+        <geometry><mesh scale="1.0 1.0 1.0" filename="${M}/tilt_ram_mount_outboard.dae"/></geometry>
+        <material name="bucket_steel"/>
+      </visual>
+      <visual>
+        <origin xyz="0.17904 -0.1 0.01199" rpy="0 0 0"/>
+        <geometry><mesh scale="1.0 1.0 1.0" filename="${M}/tilt_ram_mount_inboard.dae"/></geometry>
+        <material name="bucket_steel"/>
+      </visual>
+      <visual>
+        <origin xyz="0.18674 0 0.01399" rpy="-3.1415927 0 -1.5707963"/>
+        <geometry><mesh scale="1.0 1.0 1.0" filename="${M}/tilt_ram_bracket.dae"/></geometry>
+        <material name="bucket_dark"/>
+      </visual>
+      <!-- one box per tube, sized from the measured 750 x 40 x 20 extents -->
+      <collision name="${prefix}bucket_lift_arm_left_collision">
+        <origin xyz="0.35200 0.1 0.00000" rpy="0 0 0"/>
+        <geometry><box size="0.750 0.040 0.020"/></geometry>
+      </collision>
+      <collision name="${prefix}bucket_lift_arm_right_collision">
+        <origin xyz="0.35200 -0.1 0.00000" rpy="0 0 0"/>
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