Commit message: Port perseus-v3's bucket linkage and its ros2_control controllers
Replaces the mount-only bucket from fe29ecd with perseus-v3's current
description: the mount plus the lift arms, bucket, jaw, five rams and encoder
frames. bucket.urdf.xacro is v3's file with only the mesh path changed; the 33
meshes move under meshes/bucket/ as in v3, so the old top-level
bucket_mount.dae goes.

The Gazebo-only parts live in bucket.gazebo.xacro so the description stays a
straight copy: position controllers for the ten ram joints, a joint state
publisher for them, and the contact friction. The rams are driven by v3's
bucket_ram_follower.py, now in perseus_description as in v3, which perseus_sim
runs for payload:=bucket and view_perseus runs in viewer mode.

lift, tilt and jaw are ros2_control joints (bucket.ros2_control.xacro, on
GazeboSimSystem in the sim), driven by the controllers from v3's
payloads/config/bucket_controller.yaml (bucket_controllers.yaml here). The
bucket_controller launch argument takes the same choices and default as v3's
perseus.launch.py. The bucket shares the drive's controller_manager, because
gz_ros2_control runs one per model, but its controller is spawned into the
payloads namespace, so goals go to the same action as on the robot:
/payloads/<controller>/follow_joint_trajectory. Adds
joint_trajectory_controller to pixi.toml.

v3's linkage meshes segfaulted the Gazebo server in gz-common's Collada
polylist loader. They are Assimp exports whose VERTEX and NORMAL inputs share
offset 0; RViz reads that, gz-common does not. Each now gives NORMAL its own
offset with the index list interleaved to match; the geometry is unchanged.

Verified in the arena world: all three controllers activate, a
FollowJointTrajectory goal of lift 45, tilt -15, jaw 30 deg returns SUCCEEDED
with every joint on target, the rams track, and TF resolves base_link to
bucket_jaw.

File: src/perseus_description/urdf/perseus.urdf.xacro (robot description, xacro)
@@ -70,4 +70,5 @@
     <xacro:include filename="$(find perseus_description)/urdf/sensor_mount.urdf.xacro"/>
     <xacro:include filename="$(find perseus_description)/urdf/bucket.urdf.xacro"/>
+    <xacro:include filename="$(find perseus_description)/urdf/bucket.gazebo.xacro"/>
     <xacro:include filename="$(find perseus_description)/urdf/camera_d455_gazebo.xacro"/>
     <xacro:include filename="$(find realsense2_description)/urdf/_d455.urdf.xacro"/>
@@ -95,7 +96,10 @@
     <!-- Livox and RealSense both hang off the mast: see sensor_mount.urdf.xacro -->
     <xacro:sensor_mount prefix="${prefix}"/>
-    <!-- payload:=bucket attaches the bucket mount to the chassis; see bucket.urdf.xacro -->
+    <!-- payload:=bucket attaches the bucket to the chassis: the mount, lift arms,
+         bucket, jaw and rams (bucket.urdf.xacro, from perseus-v3), plus the Gazebo
+         ram followers (bucket.gazebo.xacro) -->
     <xacro:if value="${payload == 'bucket'}">
       <xacro:bucket prefix="${prefix}"/>
+      <xacro:bucket_gazebo prefix="${prefix}"/>
     </xacro:if>
   </xacro:macro>
